File: Adafruit Hat/Adafruit HaD Proto HAT rev A.brd (EAGLE design)
At the start: 65 x 56.5 mm, 46 parts, among them IC1 L298, IC2 DS18B20, IC3 DS18B20, IC4 DS18B20, K1 FINDER-30.22, K2 FINDER-30.22, K3 FINDER-30.22, K4 FINDER-30.22, U1 CAT24C32

Commit message: final circuit using rpi
Parts:
- removed F1, F2, F3, F4: (no value), e-sicherungen:LEITUNGSSCHUTZSCHALTER
- added F5: (no value), fuse:KS9V
Connections:
- new net N$88: F5.2, X1.1.1
- net N$28: now also F5.1; no longer F1.1, F2.1, F3.1, F4.1, X1.1.1
- net N$83: no longer F4.2
- net N$84: no longer F3.2
- net N$85: no longer F2.2
- net N$86: no longer F1.2
Changed lines of the file:
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@@
 <element name="X4" library="e-klemmen" package="KLEMME_1-3" value="" x="-99.06" y="-109.22"/>
 <element name="X5" library="e-klemmen" package="KLEMME_1-3" value="" x="-106.68" y="-109.22"/>
-<element name="F1" library="e-sicherungen" package="LEITUNGSSCHUTZSCHALTER" value="" x="-116.84" y="-116.84">
-<attribute name="HERSTELLER" value="" x="-116.84" y="-116.84" size="1.778" layer="27" display="off"/>
-<attribute name="FUNKTION" value="" x="-116.84" y="-116.84" size="1.778" layer="27" display="off"/>
-<attribute name="TYPE" value="" x="-116.84" y="-116.84" size="1.778" layer="27" display="off"/>
-</element>
-<element name="F2" library="e-sicherungen" package="LEITUNGSSCHUTZSCHALTER" value="" x="-127" y="-116.84">
-<attribute name="HERSTELLER" value="" x="-127" y="-116.84" size="1.778" layer="27" display="off"/>
-<attribute name="FUNKTION" value="" x="-127" y="-116.84" size="1.778" layer="27" display="off"/>
-<attribute name="TYPE" value="" x="-127" y="-116.84" size="1.778" layer="27" display="off"/>
-</element>
-<element name="F3" library="e-sicherungen" package="LEITUNGSSCHUTZSCHALTER" value="" x="-137.16" y="-116.84">
-<attribute name="HERSTELLER" value="" x="-137.16" y="-116.84" size="1.778" layer="27" display="off"/>
-<attribute name="FUNKTION" value="" x="-137.16" y="-116.84" size="1.778" layer="27" display="off"/>
-<attribute name="TYPE" value="" x="-137.16" y="-116.84" size="1.778" layer="27" display="off"/>
-</element>
-<element name="F4" library="e-sicherungen" package="LEITUNGSSCHUTZSCHALTER" value="" x="-147.32" y="-116.84">
-<attribute name="HERSTELLER" value="" x="-147.32" y="-116.84" size="1.778" layer="27" display="off"/>
-<attribute name="FUNKTION" value="" x="-147.32" y="-116.84" size="1.778" layer="27" display="off"/>
-<attribute name="TYPE" value="" x="-147.32" y="-116.84" size="1.778" layer="27" display="off"/>
-</element>
 <element name="IC2" library="1wire" package="TO92-" value="DS18B20" x="-154.94" y="-119.38"/>
 <element name="IC3" library="1wire" package="TO92-" value="DS18B20" x="-165.1" y="-119.38"/>
 <element name="IC4" library="1wire" package="TO92-" value="DS18B20" x="-175.26" y="-119.38"/>
 <element name="R8" library="rcl" package="0204V" value="" x="-175.26" y="-129.54"/>
+<element name="F5" library="fuse" package="KS9V" value="" x="-185.42" y="-121.92">
+<attribute name="OC_FARNELL" value="unknown" x="-185.42" y="-121.92" size="1.778" layer="27" display="off"/>
+<attribute name="MPN" value="" x="-185.42" y="-121.92" size="1.778" layer="27" display="off"/>
+<attribute name="OC_NEWARK" value="unknown" x="-185.42" y="-121.92" size="1.778" layer="27" display="off"/>
+<attribute name="MF" value="" x="-185.42" y="-121.92" size="1.778" layer="27" display="off"/>
+</element>
 </elements>
 <signals>
@@
 <contactref element="G2" pad="2"/>
 <contactref element="G1" pad="2"/>
-<contactref element="X1" pad="1.1"/>
 <contactref element="X1" pad="2.1"/>
 <contactref element="X6" pad="3.2"/>
@@
 <contactref element="X4" pad="3.2"/>
 <contactref element="X5" pad="3.2"/>
-<contactref element="F1" pad="1"/>
-<contactref element="F2" pad="1"/>
-<contactref element="F3" pad="1"/>
-<contactref element="F4" pad="1"/>
-<wire x1="-124.46" y1="-111.76" x2="-134.62" y2="-111.76" width="0" layer="19" extent="1-1"/>
-<wire x1="-114.3" y1="-111.76" x2="-124.46" y2="-111.76" width="0" layer="19" extent="1-1"/>
-<wire x1="-144.78" y1="-111.76" x2="-134.62" y2="-111.76" width="0" layer="19" extent="1-1"/>
-<wire x1="-101.6" y1="-111.76" x2="-114.3" y2="-111.76" width="0" layer="19" extent="1-1"/>
+<contactref element="F5" pad="1"/>
 <wire x1="-93.98" y1="-111.76" x2="-101.6" y2="-111.76" width="0" layer="19" extent="1-1"/>
 <wire x1="-86.36" y1="-111.76" x2="-93.98" y2="-111.76" width="0" layer="19" extent="1-1"/>
 <wire x1="-78.74" y1="-111.76" x2="-86.36" y2="-111.76" width="0" layer="19" extent="1-1"/>
-<wire x1="-10.16" y1="-38.1" x2="-78.74" y2="-111.76" width="0" layer="19" extent="1-1"/>
-<wire x1="-7.62" y1="-38.1" x2="-10.16" y2="-38.1" width="0" layer="19" extent="1-1"/>
+<wire x1="-185.42" y1="-118.11" x2="-101.6" y2="-111.76" width="0" layer="19" extent="1-1"/>
+<wire x1="-7.62" y1="-38.1" x2="-78.74" y2="-111.76" width="0" layer="19" extent="1-1"/>
 <wire x1="2.54" y1="-38.1" x2="-7.62" y2="-38.1" width="0" layer="19" extent="1-1"/>
 <wire x1="2.54" y1="-33.02" x2="2.54" y2="-38.1" width="0" layer="19" extent="1-1"/>
@@
 <signal name="N$83">
 <contactref element="K1" pad="11"/>
-<contactref element="F4" pad="2"/>
-<wire x1="-144.78" y1="-121.92" x2="1.27" y2="-49.53" width="0" layer="19" extent="1-1"/>
 </signal>
 <signal name="N$84">
 <contactref element="K2" pad="11"/>
-<contactref element="F3" pad="2"/>
-<wire x1="-134.62" y1="-121.92" x2="1.27" y2="-59.69" width="0" layer="19" extent="1-1"/>
 </signal>
 <signal name="N$85">
 <contactref element="K3" pad="11"/>
-<contactref element="F2" pad="2"/>
-<wire x1="1.27" y1="-69.85" x2="-124.46" y2="-121.92" width="0" layer="19" extent="1-1"/>
 </signal>
 <signal name="N$86">
 <contactref element="K4" pad="11"/>
-<contactref element="F1" pad="2"/>
-<wire x1="1.27" y1="-80.01" x2="-114.3" y2="-121.92" width="0" layer="19" extent="1-1"/>
 </signal>
 <signal name="1W">
@@
 <contactref element="R8" pad="1"/>
 </signal>
+<signal name="N$88">
+<contactref element="X1" pad="1.1"/>
+<contactref element="F5" pad="2"/>
+<wire x1="-10.16" y1="-38.1" x2="-185.42" y2="-125.73" width="0" layer="19" extent="1-1"/>
+</signal>
 </signals>

Commit message: improve scematic
Parts:
- removed FID2, FID3: FIDUCIAL"", microbuilder:FIDUCIAL_1MM
- removed IC2, IC3, IC4: DS18B20, 1wire:TO92-
- removed R7: (no value), e-spulen-transformatoren:SPULE
- removed R8: (no value), rcl:0204V
- added IC5, IC6, IC7: DS18B20, 1wire:TO92-
- added K5, K6, K7, K8: FINDER-30.22, relay:FINDER-30.22
- added M5: Maischepumpe, e-motoren:MOTOR_1-PHASEN
- added M6: Ruerwerk, e-motoren:MOTOR_1-PHASEN
- added OK5, OK6, OK7, OK8: 4N33, optocoupler:DIL06
- added R10, R9: Gasv., e-spulen-transformatoren:SPULE
- added S1: (no value), e-schalter:SCHLIESSER_KIPPSCHALTER
- added S3: (no value), e-schalter:AUSTASTER
- added X10, X11, X12, X13: (no value), e-klemmen:KLEMME_1-3
- added X14, X15: (no value), e-steckverbinder:STECKDOSE
- added X16, X17, X18: NC3FAV2, con-neutrik_ag:NC3FAV2
- added X8, X9: (no value), e-klemmen:KLEMME_1-2
- M1, M2: value (none) -> Pumpe
- R4, R5: value (none) -> Gasv.
- R6: device e-spulen-transformatoren:SPULE -> rcl:0204V
- moved R6 192.2 mm to (-198.1, -256.5)
Connections:
- new net N$100: K7.A1, OK7.4
- new net N$101: K8.A1, OK8.4
- new net N$102: R5.1, X9.1.1
- new net N$103: R5.2, X9.2.1
- new net N$104: K7.14, X13.1.2
- new net N$105: K8.14, X12.1.2
- new net N$106: K5.A2, K6.A2, K7.A2, K8.A2, R6.2, X16.1, X17.1, X18.1
- new net N$108: R9.1, X13.1.1
- new net N$109: R9.2, X13.3.1
- new net N$110: R10.2, X12.3.1
- new net N$111: R10.1, X12.1.1
- new net N$112: K6.14, X10.1.2
- new net N$114: K5.14, X11.1.2
- new net N$118: X13.2.1
- new net N$119: X12.2.1
- new net N$120: K5.11
- new net N$121: K6.11
- new net N$122: K7.11
- new net N$123: K8.11
- new net N$125: X15.PE, X4.2.1
- new net N$126: X14.PE, X5.2.1
- new net N$132: OK1.1, OK2.1, OK3.1, OK4.1, OK5.1, OK6.1, OK7.1, OK8.1, U$4.3.3V
- new net N$89: F5.1, S1.13
- new net N$90: S1.14, S3.11
- new net N$91: R6.1, U$4.12, X16.3, X17.3, X18.3
- new net N$92: G1.4, G2.4, K1.A2, K2.A2, K3.A2, K4.A2
- new net N$93: OK8.2, U$4.4
- new net N$94: OK7.2, U$4.5
- new net N$95: OK6.2, U$4.6
- new net N$96: OK5.2, U$4.7
- new net N$97: R1.2, R2.2, U1.8
- new net N$98: K5.A1, OK5.4
- new net N$99: K6.A1, OK6.4
- net 1W: now also IC5.2, IC6.2, IC7.2; no longer IC2.2, IC3.2, IC4.2
- net 3.3V: no longer R1.2, R2.2, U1.8
- net 5.0V: now also IC1.10, IC1.5; no longer IC1.12, IC1.7, R8.2
- net GND: now also IC1.12, IC1.7, IC5.1, IC6.1, IC7.1, X16.2, X17.2, X18.2; no longer G1.4, G2.4, IC1.10, IC1.5, IC2.1, IC3.1, IC4.1, K1.A2, K2.A2, K3.A2, K4.A2
- net N$24: now also U$4.13; no longer U$4.2
- net N$25: now also U$4.14/A0; no longer U$4.3
- net N$26: now also X8.1.2; no longer R4.1
- net N$28: now also S3.12, X10.3.2, X11.3.2, X12.3.2, X13.3.2; no longer F5.1
- net N$29: now also X8.2.1; no longer IC1.13
- net N$30: now also X9.1.2; no longer R5.1
- net N$31: now also X9.2.2; no longer R5.2
- net N$32: now also IC1.13, X8.2.2; no longer OK1.1, OK2.1, OK3.1, OK4.1, U$4.3.3V
- net N$33: now also U$4.8; no longer U$4.4
- net N$34: now also U$4.9; no longer U$4.5
- net N$35: now also U$4.10; no longer U$4.6
- net N$36: now also U$4.11; no longer U$4.7
- net N$37: now also OK5.6, OK6.6, OK7.6, OK8.6
- net N$69: now also M5.U, X14.L1
- net N$72: now also M6.U, X15.L1, X4.1.1; no longer R6.2, X5.3.1
- net N$73: now also M5.PE; no longer R7.2, X4.3.1
- net N$74: now also M6.PE; no longer X4.1.1
- net N$81: now also M6.V, X15.N, X4.3.1; no longer X5.2.1
- net N$82: now also M5.V, X14.N, X5.3.1; no longer X4.2.1
- net N$87: now also R4.1, X8.1.1; no longer R8.1
- net VDD: now also IC5.3, IC6.3, IC7.3; no longer IC2.3, IC3.3, IC4.3
Routing:
- net 3.3V: track 150.6 -> 142.5 mm
- net N$97: track 0.00 -> 2.67 mm
